File: design/kicad/solderdemon_m68k.kicad_pcb (KiCad board)
At the start: 4 copper layers, 165 x 100 mm, 87 parts, among them IC1 MC68010P10, IC15 555N, IC2 ATF1502AS-10JU44, IC3 ATF1502AS-10JU44, IC4 XR68C681CJTR-F, IC7 74LS148, J1 UART_A, J2 UART_B, J3 Conn_02x32_Odd_Even, J4 Conn_01x06, J5 PWR, J8 Conn_01x02_Male, J9 JTAG, Q1 3.6864MHz, Q2 5H8ET-10.000, U1 SST39SF040, U2 SST39SF040, U3 AS6C4008-55PCN, U4 AS6C4008-55PCN

Commit message: Optimize SolderDemon m68k r1 routing and regenerate manufacturing files
Routing:
- net A18: track 325.8 -> 215.5 mm, vias 12 -> 4
- net D6: track 344.6 -> 248.6 mm, vias 13 -> 11
